File: Hardware/GrenadeConversionV3/GrenadeConversion3.kicad_pcb (KiCad board)
At the start: 2 copper layers, 18.5 x 18 mm, 14 parts, among them J1 Grenade, J2 Programming, J3 IR_RX, U1 STM32F070CBTx

Commit message: Update HW to V3.1 - Layout changes for easier manufacturing
Other:
- rule pad_to_mask_clearance: 0.2 -> 0.0762
- board text added: "v3.1"
- board text removed: "v3.0"
Changed lines of the file:
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@@
-(kicad_pcb (version 20171130) (host pcbnew "(5.0.0)")
+(kicad_pcb (version 20171130) (host pcbnew "(5.1.2)-2")
   (general
     (thickness 1.6)
@@
     (zone_45_only no)
     (trace_min 0.1524)
-    (segment_width 0.127)
-    (edge_width 0.15)
     (via_size 0.6)
     (via_drill 0.4)
@@
     (uvia_min_size 0.2)
     (uvia_min_drill 0.1)
-    (pcb_text_width 0.3)
-    (pcb_text_size 0.127 1.5)
+    (edge_width 0.15)
+    (segment_width 0.127)
+    (pcb_text_width 0.0508)
+    (pcb_text_size 0.2032 1.5)
     (mod_edge_width 0.15)
     (mod_text_size 0.762 0.762)
@@
     (pad_size 1.524 1.524)
     (pad_drill 0.762)
-    (pad_to_mask_clearance 0.2)
+    (pad_to_mask_clearance 0.0762)
     (aux_axis_origin 0 0)
     (visible_elements 7FFFFFFF)
@@
     (descr "48 LEAD LQFP 7x7mm (see MICREL LQFP7x7-48LD-PL-1.pdf)")
     (tags "QFP 0.5")
+    (solder_mask_margin 0.0508)
     (attr smd)
     (fp_text reference U1 (at -4.29 -4.35) (layer F.SilkS)
@@
     (effects (font (size 0.508 0.508) (thickness 0.127)))
   )
-  (gr_text v3.0 (at 108.84408 100.3554) (layer F.SilkS)
+  (gr_text v3.1 (at 108.84408 100.3554) (layer F.SilkS)
     (effects (font (size 0.889 0.889) (thickness 0.127)))
   )
@@
   (segment (start 120.4722 98.8402) (end 119.676 98.044) (width 0.254) (layer B.Cu) (net 2))
   (segment (start 120.4722 99.822) (end 120.4722 98.8402) (width 0.254) (layer B.Cu) (net 2))
-  (segment (start 113.112 98.254) (end 113.449 97.917) (width 0.254) (layer F.Cu) (net 2))
-  (segment (start 112.208 98.254) (end 113.112 98.254) (width 0.254) (layer F.Cu) (net 2))
-  (via (at 113.587977 97.923977) (size 0.6) (drill 0.4) (layers F.Cu B.Cu) (net 2))
-  (segment (start 113.449 97.917) (end 113.581 97.917) (width 0.254) (layer F.Cu) (net 2))
-  (segment (start 113.581 97.917) (end 113.587977 97.923977) (width 0.254) (layer F.Cu) (net 2))
   (segment (start 113.287978 98.223976) (end 113.587977 97.923977) (width 0.254) (layer B.Cu) (net 2))
   (segment (start 112.268 99.243954) (end 113.287978 98.223976) (width 0.254) (layer B.Cu) (net 2))
@@
   (segment (start 115.42268 89.9354) (end 115.5506 90.06332) (width 0.254) (layer B.Cu) (net 2))
   (segment (start 115.5506 90.06332) (end 119.01932 90.06332) (width 0.254) (layer B.Cu) (net 2))
+  (via (at 112.2934 98.9838) (size 0.6) (drill 0.4) (layers F.Cu B.Cu) (net 2))
+  (segment (start 112.208 98.254) (end 112.208 98.8984) (width 0.254) (layer F.Cu) (net 2))
+  (segment (start 112.208 98.8984) (end 112.2934 98.9838) (width 0.254) (layer F.Cu) (net 2))
+  (segment (start 112.268 99.0092) (end 112.268 99.243954) (width 0.254) (layer B.Cu) (net 2))
+  (segment (start 112.2934 98.9838) (end 112.268 99.0092) (width 0.254) (layer B.Cu) (net 2))
   (segment (start 109.3156 102.108) (end 108.204 102.108) (width 0.1524) (layer B.Cu) (net 3))
   (segment (start 110.068 102.108) (end 109.3156 102.108) (width 0.1524) (layer B.Cu) (net 3))
